File: 01-three-band-EQ/design/KicadDesign/KicadDesign.kicad_sch (KiCad schematic)
At the start: 29 parts, among them J1 Supply, J2 Output, J3 Input, U1 TL072, U2 TL072, U3 TL072

Commit message: Kicad corregido
Parts:
- added unit 2 of U3
Connections:
- net IN: now also U3.6 (-), U3.7; no longer J3.1 (Pin_1)
- new net INPUT: J3.1 (Pin_1), U3.5 (+)
Other:
- moved on the sheet: J3
Changed lines of the file:
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@@
 	(wire
 		(pts
+			(xy 28.448 57.658) (xy 28.448 59.944)
+		)
+		(stroke
+			(width 0)
+			(type default)
+		)
+	)
+	(wire
+		(pts
 			(xy 68.58 87.63) (xy 68.58 97.79)
 		)
@@
 	(wire
 		(pts
+			(xy 28.448 69.85) (xy 43.688 69.85)
+		)
+		(stroke
+			(width 0)
+			(type default)
+		)
+	)
+	(wire
+		(pts
 			(xy 73.66 114.3) (xy 85.09 114.3)
 		)
@@
 	(wire
 		(pts
+			(xy 43.688 69.85) (xy 43.688 62.484)
+		)
+		(stroke
+			(width 0)
+			(type default)
+		)
+	)
+	(wire
+		(pts
 			(xy 45.72 127) (xy 49.53 127)
 		)
@@
 	(wire
 		(pts
+			(xy 28.448 65.024) (xy 28.448 69.85)
+		)
+		(stroke
+			(width 0)
+			(type default)
+		)
+	)
+	(wire
+		(pts
 			(xy 150.876 55.372) (xy 155.448 55.372)
 		)
@@
 	)
 	(label "IN"
+		(at 43.688 62.484 0)
+		(effects
+			(font
+				(size 1.27 1.27)
+			)
+			(justify left bottom)
+		)
+	)
+	(label "IN"
 		(at 86.36 129.54 0)
 		(effects
@@
 		)
 	)
+	(label "INPUT"
+		(at 28.448 57.658 0)
+		(effects
+			(font
+				(size 1.27 1.27)
+			)
+			(justify left bottom)
+		)
+	)
 	(label "OUT_BP"
 		(at 148.59 132.08 0)
@@
 		)
 	)
-	(label "IN"
-		(at 24.13 59.944 0)
+	(label "INPUT"
+		(at 20.066 59.944 0)
 		(effects
 			(font
@@
 	(symbol
 		(lib_id "power:GND")
-		(at 24.13 62.484 0)
+		(at 20.066 62.484 0)
 		(unit 1)
 		(body_style 1)
@@
 		(dnp no)
 		(property "Reference" "#PWR015"
-			(at 24.13 68.834 0)
+			(at 20.066 68.834 0)
 			(hide yes)
 			(show_name no)
@@
 		)
 		(property "Value" "GND"
-			(at 24.13 80.264 0)
+			(at 20.066 80.264 0)
 			(show_name no)
 			(do_not_autoplace no)
@@
 		)
 		(property "Footprint" ""
-			(at 24.13 62.484 0)
+			(at 20.066 62.484 0)
 			(hide yes)
 			(show_name no)
@@
 		)
 		(property "Datasheet" ""
-			(at 24.13 62.484 0)
+			(at 20.066 62.484 0)
 			(hide yes)
 			(show_name no)
@@
 		)
 		(property "Description" "Power symbol creates a global label with name \"GND\" , ground"
-			(at 24.13 62.484 0)
+			(at 20.066 62.484 0)
 			(hide yes)
 			(show_name no)
@@
 	)
 	(symbol
+		(lib_id "Amplifier_Operational:TL072")
+		(at 36.068 62.484 0)
+		(unit 2)
+		(body_style 1)
+		(exclude_from_sim no)
+		(in_bom yes)
+		(on_board yes)
+		(in_pos_files yes)
+		(dnp no)
+		(fields_autoplaced yes)
+		(property "Reference" "U3"
+			(at 36.068 52.832 0)
+			(show_name no)
+			(do_not_autoplace no)
+			(effects
+				(font
+					(size 1.27 1.27)
+				)
+			)
+		)
+		(property "Value" "TL072"
+			(at 36.068 55.372 0)
+			(show_name no)
+			(do_not_autoplace no)
+			(effects
+				(font
+					(size 1.27 1.27)
+				)
+			)
+		)
+		(property "Footprint" "Package_DIP:DIP-8_W7.62mm_LongPads"
+			(at 36.068 62.484 0)
+			(hide yes)
+			(show_name no)
+			(do_not_autoplace no)
+			(effects
+				(font
+					(size 1.27 1.27)
+				)
+			)
+		)
+		(property "Datasheet" "http://www.ti.com/lit/ds/symlink/tl071.pdf"
+			(at 36.068 62.484 0)
+			(hide yes)
+			(show_name no)
+			(do_not_autoplace no)
+			(effects
+				(font
+					(size 1.27 1.27)
+				)
+			)
+		)
+		(property "Description" "Dual Low-Noise JFET-Input Operational Amplifiers, DIP-8/SOIC-8"
+			(at 36.068 62.484 0)
+			(hide yes)
+			(show_name no)
+			(do_not_autoplace no)
+			(effects
+				(font
+					(size 1.27 1.27)
+				)
+			)
+		)
+		(pin "3"
+		)
+		(pin "1"
+		)
+		(pin "6"
+		)
+		(pin "5"
+		)
+		(pin "4"
+		)
+		(pin "2"
+		)
+		(pin "7"
+		)
+		(pin "8"
+		)
+		(instances
+			(project "KicadDesign"
+				(path "/c1a351fa-3a02-49bc-9f68-a75d5503bf21"
+					(reference "U3")
+					(unit 2)
+				)
+			)
+		)
+	)
+	(symbol
 		(lib_id "Device:C")
 		(at 58.42 44.45 180)
@@
 	(symbol
 		(lib_id "Connector:Conn_01x02_Pin")
-		(at 19.05 59.944 0)
+		(at 14.986 59.944 0)
 		(unit 1)
 		(body_style 1)
@@
 		(fields_autoplaced yes)
 		(property "Reference" "J3"
-			(at 19.685 54.356 0)
+			(at 15.621 54.356 0)
 			(show_name no)
 			(do_not_autoplace no)
@@
 		)
 		(property "Value" "Input"
-			(at 19.685 56.896 0)
+			(at 15.621 56.896 0)
 			(show_name no)
 			(do_not_autoplace no)
@@
 		)
 		(property "Footprint" "TerminalBlock:TerminalBlock_MaiXu_MX126-5.0-02P_1x02_P5.00mm"
-			(at 19.05 59.944 0)
+			(at 14.986 59.944 0)
 			(hide yes)
 			(show_name no)
@@
 		)
 		(property "Datasheet" ""
-			(at 19.05 59.944 0)
+			(at 14.986 59.944 0)
 			(hide yes)
 			(show_name no)
@@
 		)
 		(property "Description" "Generic connector, single row, 01x02, script generated"
-			(at 19.05 59.944 0)
+			(at 14.986 59.944 0)
 			(hide yes)
 			(show_name no)

Commit message: Placa routeada nomas faltan 2 PINES, voy a seguir intentando pero si no con cables
Parts:
- removed J1: Supply, TerminalBlock:TerminalBlock_MaiXu_MX126-5.0-02P_1x02_P5.00mm, symbol Connector:Conn_01x02_Pin
- added J4: Supply, TerminalBlock:TerminalBlock_MaiXu_MX126-5.0-03P_1x03_P5.00mm, symbol Connector:Conn_01x03_Pin
- added R13: 12k, Resistor_THT:R_Axial_DIN0411_L9.9mm_D3.6mm_P5.08mm_Vertical, symbol Device:R
- added R14: 1k, Resistor_THT:R_Axial_DIN0411_L9.9mm_D3.6mm_P5.08mm_Vertical, symbol Device:R
- added RV4: 1k, Potentiometer_THT:Potentiometer_Alps_RK163_Single_Horizontal, symbol Device:R_Potentiometer
- R1, R10, R11, R2, R3, R4, R5, R6, R7, R8, R9: footprint Resistor_THT:R_Axial_DIN0309_L9.0mm_D3.2mm_P15.24mm_Horizontal -> Resistor_THT:R_Axial_DIN0411_L9.9mm_D3.6mm_P5.08mm_Vertical
- R12: value 2.7k -> 1.5k; footprint Resistor_THT:R_Axial_DIN0309_L9.0mm_D3.2mm_P15.24mm_Horizontal -> Resistor_THT:R_Axial_DIN0411_L9.9mm_D3.6mm_P5.08mm_Vertical
Connections:
- net GND: now also J4.2 (Pin_2), R14.2
- net Out: now also R13.1, R14.1; no longer R12.1, U3.1
- net VCC: now also J4.1 (Pin_1)
- net VEE: now also J4.3 (Pin_3)
- net at R10.1, R11.1, R9.1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: now also RV4.1; no longer R12.2
- new net: R12.1, R13.2, U3.1
- new net: R12.2, RV4.2, RV4.3
Other:
- moved on the sheet: J2, R12

Commit message: Placa routeada porfavor checar
Parts:
- added R15: 0, Resistor_THT:R_Axial_DIN0411_L9.9mm_D3.6mm_P5.08mm_Vertical, symbol Device:R
- added R16: 270k, Resistor_THT:R_Axial_DIN0207_L6.3mm_D2.5mm_P15.24mm_Horizontal, symbol Device:R
Connections:
- net IN: now also R16.1, R16.2
- net VEE: now also R15.1, R15.2

Commit message: feat: PCB routed
Parts:
- removed R15: 0, Resistor_THT:R_Axial_DIN0411_L9.9mm_D3.6mm_P5.08mm_Vertical, symbol Device:R
- removed R16: 270k, Resistor_THT:R_Axial_DIN0207_L6.3mm_D2.5mm_P15.24mm_Horizontal, symbol Device:R
- C7: footprint Capacitor_THT:C_Disc_D5.0mm_W2.5mm_P2.50mm -> Capacitor_THT:C_Disc_D8.0mm_W5.0mm_P7.50mm
- R1, R3: footprint Resistor_THT:R_Axial_DIN0411_L9.9mm_D3.6mm_P5.08mm_Vertical -> Resistor_THT:R_Axial_DIN0411_L9.9mm_D3.6mm_P12.70mm_Horizontal
Connections:
- net OUT_HP: now also RV3.1
- net OUT_LP: no longer RV3.1
Other:
- moved on the sheet: U3B

Commit message: feat: PCB routed
Connections:
- net GND: now also J3.1 (Pin_1); no longer J3.2 (Pin_2)
- net INPUT: now also J3.2 (Pin_2); no longer J3.1 (Pin_1)
- net VCC: now also J4.3 (Pin_3); no longer J4.1 (Pin_1)
- net VEE: now also J4.1 (Pin_1); no longer J4.3 (Pin_3)
Other:
- moved on the sheet: J3
