File: 01-three-band-EQ/design/KicadDesign/KicadDesign.kicad_sch (KiCad schematic)
At the start: 32 parts, among them J2 Output, J3 Input, J4 Supply, U1 TL072, U2 TL072, U3 TL072

Commit message: fix: rm IN duplicate trace
Connections:
- net IN: no longer C6.2, C7.2, U1.1, U1.2 (-)
- new net: C6.2, C7.2, U1.1, U1.2 (-)
Changed lines of the file:
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@@
-		)
-	)
-	(label "IN"
-		(at 86.36 129.54 0)
-		(effects
-			(font
-				(size 1.27 1.27)
-			)
-			(justify left bottom)
 		)
 	)
