File: 01-three-band-EQ/design/KicadDesign/_restore_backup_2026-10-07T10-02-39-528/KicadDesign.kicad_pcb (KiCad board)
At the start: 2 copper layers, 96 x 60 mm, 32 parts, among them J2 Output, J3 Input, J4 Supply, U1 TL072, U2 TL072, U3 TL072

Commit message: feat: Add ground plane
Parts:
- C1, C2, C3, C4, C6, C8: footprint Capacitor_THT:C_Disc_D5.0mm_W2.5mm_P5.00mm -> Capacitor_THT:C_Disc_D5.0mm_W2.5mm_P2.50mm
- C5: footprint Capacitor_THT:C_Disc_D8.0mm_W5.0mm_P7.50mm -> Capacitor_THT:C_Disc_D5.0mm_W2.5mm_P2.50mm
- C7: footprint Capacitor_THT:C_Disc_D5.0mm_W2.5mm_P5.00mm -> Capacitor_THT:C_Disc_D8.0mm_W5.0mm_P7.50mm
- R1, R3: footprint Resistor_THT:R_Axial_DIN0207_L6.3mm_D2.5mm_P10.16mm_Horizontal -> Resistor_THT:R_Axial_DIN0411_L9.9mm_D3.6mm_P12.70mm_Horizontal
- moved R4 3.78 mm to (59.7, 66.6)
- moved R1 2.65 mm to (31.4, 83.3)
- moved C4 1.94 mm to (86.5, 63.1)
- moved R3 1.50 mm to (46.9, 88.4)
- moved C7 1.09 mm to (80.6, 87.6)
- moved C5 0.81 mm to (64.2, 75.5)
- moved C3 0.79 mm to (59.6, 78.1), turned to 90 degrees
- turned C2 to 90 degrees
Routing:
- net /IN: track 131.8 -> 139.7 mm
- net VCC: track 145.6 -> 141.4 mm
- net Net-(U2A-+): track 11.8 -> 14.9 mm
- net Net-(C1-Pad1): track 13.1 -> 15.8 mm
- net /OUT_LP: track 38.9 -> 41.4 mm
- net Net-(U2B-+): track 17.4 -> 15.2 mm
- net GND: track 203.5 -> 205.5 mm
- net Net-(C7-Pad1): track 16.1 -> 17.6 mm
- removed copper zone on B.Cu, net GND
Other:
- board size 96 x 60 mm -> 96.5 x 60 mm
